Commit message: ikpy

File: robo.urdf (robot description, URDF)
Before this commit: robot robo, 4 links, 4 joints
Links:
- added link arm3; visual box size=0.017 0.017 0.07
- added link top; visual cylinder length=0.045 radius=0.04
- link arm1: geometry visual cylinder length=0.120 radius=0.022
- link arm2: geometry visual cylinder length=0.120 radius=0.0175
- link base_link: geometry visual cylinder length=0.015 radius=0.089
- link base_rot: geometry visual box size=0.05 0.05 0.1
Joints:
- removed joint elbow_joint
- removed joint rot_joint
- removed joint shoulder_joint
- added joint arm1_joint: type revolute, parent base_rot, child arm1, origin xyz=0 0 0.05 rpy=0 0 0, axis 1 0 0, limit lower=-1.57 upper=1.57
- added joint arm2_joint: type revolute, parent arm1, child arm2, origin xyz=0 0 0.120 rpy=0 0 0, axis 1 0 0, limit lower=-1.57 upper=1.57
- added joint arm3_joint: type revolute, parent arm2, child arm3, origin xyz=0 0 0.12 rpy=0 0 0, axis 1 0 0, limit lower=-1.57 upper=1.57
- added joint top_joint: type revolute, parent arm3, child top, origin xyz=0 0 0.045 rpy=0 0 0, axis -1 0 0, limit lower=-1.57 upper=1.57
- joint base_joint: axis 0 0 -1 -> 0 0 1; origin xyz=0 0 0.072 rpy=0 0 0 -> xyz=0 0 0.065 rpy=0 0 0

Commit message: ikpy

File: robo.urdf (robot description, URDF)
Before this commit: robot robot_arm, 6 links, 5 joints
Links:
- removed link top
Joints:
- removed joint top_joint
- joint arm2_joint: limit lower=-1.57 upper=1.57 -> lower=-3.14 upper=0.01
- joint arm3_joint: axis 1 0 0 -> -1 0 0
- joint base_joint: axis 0 0 1 -> 0 0 -1
